File: hardware/kicad/navdim/navdim.kicad_pcb (KiCad board)
At the start: 2 copper layers, 65 x 18 mm, 22 parts, among them J1 Screw_Terminal_01x02, J2 Conn_01x06_Male, J3 Screw_Terminal_01x02, Q1 DMN2055U, SW1 SW_Push, SW2 Rotary_Encoder_Switch, U1 L78L33_SOT89, U2 MSP430FR2433RGE

Commit message: Basic PCB layout
Parts:
- moved GND 8.14 mm to (143.3, 123.6), turned to 0 degrees
- moved TST 7.13 mm to (150.9, 123.6), turned to 0 degrees
- moved 3v3 3.09 mm to (145.8, 123.6), turned to 0 degrees
- moved C3 2.54 mm to (150.8, 111.3)
- moved C4 2.54 mm to (149.1, 111.3)
- moved RST 2.09 mm to (148.3, 123.6), turned to 0 degrees
- moved R1 1.51 mm to (156.2, 122.8)
- moved R3 1.41 mm to (155.8, 116.2)
- moved C5 1.32 mm to (158.8, 122.8)
- moved D1 0.82 mm to (152.2, 116.2)
- turned U2 to 0 degrees
Connections:
- U2 pad 25: (no net) -> GND
- U2 pad 8: PLAMP -> PLED
- U2 pad 9: PLED -> PLAMP
Routing:
- net PLAMP: track 1.94 -> 34.4 mm
- net GND: track 77.2 -> 107.8 mm, vias 0 -> 9
- net pRotaryButton: track 0.00 -> 22.0 mm
- net RST: track 42.5 -> 61.1 mm
- net TEST: track 0.00 -> 17.8 mm
- net RXD: track 0.00 -> 13.2 mm
- net TXD: track 0.00 -> 9.91 mm
- net +3V3: track 33.6 -> 41.7 mm
- net pRotary2: track 14.9 -> 11.6 mm
- net PLED: track 0.00 -> 2.04 mm
- net Net-(D1-Pad2): track 0.00 -> 1.76 mm
- net pRotary1: track 5.90 -> 4.23 mm
- net VCC: track 71.6 -> 72.9 mm
- added copper zone on B.Cu, net GND
Other:
- rule pad_to_mask_clearance: 0.05 -> 0
- board text added: "navdim v1.0 www.birchavenue.org"
