File: hardware/kicad/navdim/navdim.sch (KiCad schematic (older format))
At the start: 22 parts, among them J1 Screw_Terminal_01x02, J2 Conn_01x06_Male, J3 Screw_Terminal_01x02, Q1 DMN2055U, SW1 SW_Push, SW2 Rotary_Encoder_Switch, U1 L78L33_SOT89, U2 MSP430FR2433RGE

Commit message: Basic PCB layout
Parts:
- 3v3: renamed from TP3; footprint TestPoint:TestPoint_Pad_D2.0mm -> TestPoint:TestPoint_Pad_D1.5mm
- GND: renamed from TP4; footprint TestPoint:TestPoint_Pad_D2.0mm -> TestPoint:TestPoint_Pad_D1.5mm
- RST: renamed from TP2; footprint TestPoint:TestPoint_Pad_D2.0mm -> TestPoint:TestPoint_Pad_D1.5mm
- TST: renamed from TP1; footprint TestPoint:TestPoint_Pad_D2.0mm -> TestPoint:TestPoint_Pad_D1.5mm
Connections:
- net GND: now also U2.25 (VSS)
- net PLAMP: now also U2.9 (P1.2/UCB0SIMO/UCB0SDA/TA0.2/A2/Veref); no longer U2.8 (P1.1/UCB0CLK/TA0.1/A1)
- net PLED: now also U2.8 (P1.1/UCB0CLK/TA0.1/A1); no longer U2.9 (P1.2/UCB0SIMO/UCB0SDA/TA0.2/A2/Veref)
Changed lines of the file:
@@
 PLAMP
 Text GLabel 4550 4000 0    50   Input ~ 0
+PLED
+Text GLabel 4550 4100 0    50   Input ~ 0
 PLAMP
-Text GLabel 4550 4100 0    50   Input ~ 0
-PLED
 NoConn ~ 4550 4300
 NoConn ~ 4550 4200
@@
 PLED
 $Comp
-L Connector:TestPoint TP1
+L Connector:TestPoint TST
 U 1 1 61767A30
 P 7450 1850
-F 0 "TP1" V 7450 2050 50  0000 L CNN
+F 0 "TST" V 7450 2050 50  0000 L CNN
 F 1 "TestPoint" V 7450 1100 50  0001 L CNN
-F 2 "TestPoint:TestPoint_Pad_D2.0mm" H 7650 1850 50  0001 C CNN
+F 2 "TestPoint:TestPoint_Pad_D1.5mm" H 7650 1850 50  0001 C CNN
 F 3 "~" H 7650 1850 50  0001 C CNN
 	1    7450 1850
@@
 $EndComp
 $Comp
-L Connector:TestPoint TP2
+L Connector:TestPoint RST
 U 1 1 61767D78
 P 7450 2000
-F 0 "TP2" V 7450 2250 50  0000 C CNN
+F 0 "RST" V 7450 2250 50  0000 C CNN
 F 1 "TestPoint" H 7508 2027 50  0001 L CNN
-F 2 "TestPoint:TestPoint_Pad_D2.0mm" H 7650 2000 50  0001 C CNN
+F 2 "TestPoint:TestPoint_Pad_D1.5mm" H 7650 2000 50  0001 C CNN
 F 3 "~" H 7650 2000 50  0001 C CNN
 	1    7450 2000
@@
 $EndComp
 $Comp
-L Connector:TestPoint TP3
+L Connector:TestPoint 3v3
 U 1 1 61768157
 P 7450 2150
-F 0 "TP3" V 7450 2350 50  0000 L CNN
+F 0 "3v3" V 7450 2350 50  0000 L CNN
 F 1 "TestPoint" H 7508 2177 50  0001 L CNN
-F 2 "TestPoint:TestPoint_Pad_D2.0mm" H 7650 2150 50  0001 C CNN
+F 2 "TestPoint:TestPoint_Pad_D1.5mm" H 7650 2150 50  0001 C CNN
 F 3 "~" H 7650 2150 50  0001 C CNN
 	1    7450 2150
@@
 $EndComp
 $Comp
-L Connector:TestPoint TP4
+L Connector:TestPoint GND
 U 1 1 617684AC
 P 7450 2300
-F 0 "TP4" V 7450 2550 50  0000 C CNN
+F 0 "GND" V 7450 2550 50  0000 C CNN
 F 1 "TestPoint" H 7508 2327 50  0001 L CNN
-F 2 "TestPoint:TestPoint_Pad_D2.0mm" H 7650 2300 50  0001 C CNN
+F 2 "TestPoint:TestPoint_Pad_D1.5mm" H 7650 2300 50  0001 C CNN
 F 3 "~" H 7650 2300 50  0001 C CNN
 	1    7450 2300
@@
 	1    0    0    -1
 $EndComp
+$Comp
+L power:GND #PWR0119
+U 1 1 6173ABA5
+P 5350 4550
+F 0 "#PWR0119" H 5350 4300 50  0001 C CNN
+F 1 "GND" H 5355 4377 50  0000 C CNN
+F 2 "" H 5350 4550 50  0001 C CNN
+F 3 "" H 5350 4550 50  0001 C CNN
+	1    5350 4550
+	1    0    0    -1
+$EndComp

Commit message: update
Parts:
- renumbered GND to GND1, RST to RST1, TST to TST1
Changed lines of the file:
@@
 PLED
 $Comp
-L Connector:TestPoint TST
+L Connector:TestPoint TST1
 U 1 1 61767A30
 P 7450 1850
-F 0 "TST" V 7450 2050 50  0000 L CNN
+F 0 "TST1" V 7450 2050 50  0000 L CNN
 F 1 "TestPoint" V 7450 1100 50  0001 L CNN
 F 2 "TestPoint:TestPoint_Pad_D1.5mm" H 7650 1850 50  0001 C CNN
@@
 $EndComp
 $Comp
-L Connector:TestPoint RST
+L Connector:TestPoint RST1
 U 1 1 61767D78
 P 7450 2000
-F 0 "RST" V 7450 2250 50  0000 C CNN
+F 0 "RST1" V 7450 2250 50  0000 C CNN
 F 1 "TestPoint" H 7508 2027 50  0001 L CNN
 F 2 "TestPoint:TestPoint_Pad_D1.5mm" H 7650 2000 50  0001 C CNN
@@
 $EndComp
 $Comp
-L Connector:TestPoint GND
+L Connector:TestPoint GND1
 U 1 1 617684AC
 P 7450 2300
-F 0 "GND" V 7450 2550 50  0000 C CNN
+F 0 "GND1" V 7450 2550 50  0000 C CNN
 F 1 "TestPoint" H 7508 2327 50  0001 L CNN
 F 2 "TestPoint:TestPoint_Pad_D1.5mm" H 7650 2300 50  0001 C CNN
